File: Glass_Stand_v0.2/Glass_Stand_v0.2.kicad_sch (KiCad schematic)
At the start: 33 parts, among them J1 BAT IN 12V, J2 CHARGER, J3 LED, J4 LOCK, J5 ALARM, J6 PROG, Q1 LR024N, Q2 LR024N, Q3 LR024N, SW1 SW_Push, SW2 SW_Push, U1 ESP32-WROOM-32, U2 DHT11, U3 GY-521, U4 R503_Fingerprint, U5 TB6612FNG, U6 DC-DC

Commit message: Add few passive elements to increase stability. Changed schematic size from A4 to A3.
Parts:
- removed C1, C2: 0.1uF, symbol Device:C
- removed J1: BAT IN 12V, symbol Connector:Screw_Terminal_01x02
- removed J2: CHARGER, symbol Connector:Screw_Terminal_01x02
- removed J3: LED, symbol Connector:Screw_Terminal_01x03
- removed J4: LOCK, symbol Connector:Screw_Terminal_01x02
- removed J5: ALARM, symbol Connector:Screw_Terminal_01x02
- removed J6: PROG, symbol Connector:Conn_01x03_Female
- removed Q1, Q2, Q3: LR024N, Package_DirectFET:DirectFET_MX, symbol Transistor_FET:IRF6716M
- removed R1, R10, R2, R6, R8: 11K, symbol Device:R
- removed R3, R4: 3K, symbol Device:R
- removed R5, R7, R9: 100, symbol Device:R
- removed SW1, SW2: SW_Push, symbol Switch:SW_Push
- removed U2: DHT11, Sensor:Aosong_DHT11_5.5x12.0_P2.54mm, symbol User:DHT11_user
- removed U3: GY-521, GY-521, symbol GY-521:GY-521
- removed U4: R503_Fingerprint, symbol User:R503_Fingerprint
- removed U5: TB6612FNG, symbol User:TB6612FNG
- removed U6: DC-DC, symbol User:Impulse_DC_DC
- added C?: 100uF, symbol Device:C_Polarized
- added C? (x2): 0.1uF, symbol Device:C
- added C?: 16V 100uF, symbol Device:C_Polarized
- added D? (x2): D, symbol Device:D
- added D?: D, symbol Device:D_Schottky
- added J?: BAT IN 12V, symbol Connector:Screw_Terminal_01x02
- added J?: ALARM, symbol Connector:Screw_Terminal_01x02
- added J?: LOCK, symbol Connector:Screw_Terminal_01x02
- added J?: LED, symbol Connector:Screw_Terminal_01x03
- added J?: PROG, symbol Connector:Conn_01x03_Female
- added J?: CHARGER, symbol Connector:Screw_Terminal_01x02
- added J?: SW_RST, symbol Connector:Conn_01x02_Male
- added Q? (x2): 2N7000, Package_TO_SOT_THT:TO-92_Inline, symbol Transistor_FET:2N7000
- added Q? (x2): LR024N, Package_DirectFET:DirectFET_MX, symbol Transistor_FET:IRF6716M
- added Q?: IRF4905, Package_TO_SOT_THT:TO-220-3_Vertical, symbol Transistor_FET:IRF4905
- added R? (x7): 11K, symbol Device:R
- added R?: 390K, symbol Device:R
- added R? (x3): 100, symbol Device:R
- added R?: 91K, symbol Device:R
- added SW?: SW_Push, symbol Switch:SW_Push
- added U?: DHT11, Sensor:Aosong_DHT11_5.5x12.0_P2.54mm, symbol Sensor:DHT11
- added U?: R503_Fingerprint, symbol User:R503_Fingerprint
- added U?: DC-DC, symbol User:Impulse_DC_DC
- added U?: GY-521, GY-521, symbol GY-521:GY-521
- added U?: TB6612FNG, symbol User:TB6612FNG
Connections:
- net +12V: now also C?.1, C?.1, D?.1 (K), D?.2 (A), J?.2 (Pin_2), J?.2 (Pin_2), J?.2 (Pin_2), J?.2 (Pin_2), Q?.3 (S), R?.1, R?.2, R?.2, U?.VM
- net +3V3: now also D?.1 (K), Q?.2 (G), R?.2, R?.2, U?. (OUT-), U?.1 (VCC), U?.1 (VCC), U?.6 (VCC_TOUCH), U?.STBY, U?.VCC, U?.VCC
- net GNDD: now also C?.1, C?.2, C?.2, C?.2, J?.1 (Pin_1), J?.1 (Pin_1), J?.1 (Pin_1), J?.1 (Pin_1), J?.2 (Pin_2), Q?.1 (S), Q?.3 (S), Q?.3 (S), R?.2, R?.2, R?.2, R?.2, SW?.1, U?. (OUT-), U?.2 (GND), U?.4 (GND), U?.GND, U?.GND
- net RX0: now also J?.3 (Pin_3)
- net TX0: now also J?.2 (Pin_2)
- net aSCL: now also U?.SCL
- net aSDA: now also U?.SDA
- net fingerRX: now also U?.4 (RXD)
- net fingerTX: now also U?.3 (TXD)
- net outM1: now also U?.A01
- net outM2: now also U?.A02
- net pinAlarm: now also R?.2
- net pinBatt: now also C?.1, R?.1, R?.2
- net pinDHT: now also R?.1, U?.2 (IO)
- net pinFWake: now also U?.5 (WAKEUP)
- net pinLED: now also J?.2 (Pin_2), Q?.3 (D), R?.1
- net pinLEDOn: now also R?.2
- net pinLock: now also R?.2
- net pinMDir1: now also U?.AI1
- net pinMDir2: now also U?.AI2
- net pinMPWM: now also U?.PWMA
- net swBOOT: now also J?.1 (Pin_1)
- net swRST: now also C?.2, SW?.2
- net pinLEDLow: now reaches U1.13 (IO14)
- net pinLEDLow: now also D?.2 (A), Q?.1 (S), R?.1
- new net: Q?.2 (G), R?.1, R?.1 (x3)
- new net: Q?.1 (G), Q?.3 (D), R?.1
- new net: J?.1 (Pin_1), Q?.1 (D)
- new net: D?.2 (A), J?.1 (Pin_1), Q?.1 (D)
- new net: D?.1 (K), U?. (OUT-)
- new net: J?.3 (Pin_3), Q?.2 (D)
Other:
- note added: "MCU"
- note added: "Programming Port"
- note removed: "3.3V DC"
- note removed: "ESP32"
- note removed: "Programming port"
- moved on the sheet: C3, C4, C5, R11, U1
